File: hardware/SRAM_interface/SRAM_interface.kicad_sch (KiCad schematic)
At the start: 6 parts, among them J1 FPGA_GPIO, J2 SRAM, U1 SN74LVC245APW, U2 SN74LVC245APW, U3 SN74LVC245APW, U4 SN74LVC245APW

Commit message: final commit?
Parts:
- added C1: C, symbol Device:C
Connections:
- net +3V3: now also C1.1
- net GND: now also C1.2
Changed lines of the file:
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@@
 		)
 	)
+	(junction
+		(at 150.114 118.618)
+		(diameter 0)
+		(color 0 0 0 0)
+	)
 	(no_connect
 		(at 38.862 128.778)
@@
 	(wire
 		(pts
+			(xy 150.114 118.618) (xy 150.114 118.872)
+		)
+		(stroke
+			(width 0)
+			(type default)
+		)
+	)
+	(wire
+		(pts
 			(xy 161.036 96.012) (xy 150.368 96.012)
 		)
@@
 	(wire
 		(pts
-			(xy 150.114 117.348) (xy 150.114 118.872)
+			(xy 150.114 117.348) (xy 150.114 118.618)
 		)
 		(stroke
@@
 	(symbol
 		(lib_id "power:GND")
+		(at 150.114 126.238 0)
+		(unit 1)
+		(exclude_from_sim no)
+		(in_bom yes)
+		(on_board yes)
+		(dnp no)
+		(property "Reference" "#PWR027"
+			(at 150.114 132.588 0)
+			(effects
+				(font
+					(size 1.27 1.27)
+				)
+				(hide yes)
+			)
+		)
+		(property "Value" "GND"
+			(at 150.114 129.794 0)
+			(effects
+				(font
+					(size 1.27 1.27)
+				)
+				(hide yes)
+			)
+		)
+		(property "Footprint" ""
+			(at 150.114 126.238 0)
+			(effects
+				(font
+					(size 1.27 1.27)
+				)
+				(hide yes)
+			)
+		)
+		(property "Datasheet" ""
+			(at 150.114 126.238 0)
+			(effects
+				(font
+					(size 1.27 1.27)
+				)
+				(hide yes)
+			)
+		)
+		(property "Description" "Power symbol creates a global label with name \"GND\" , ground"
+			(at 150.114 126.238 0)
+			(effects
+				(font
+					(size 1.27 1.27)
+				)
+				(hide yes)
+			)
+		)
+		(pin "1"
+		)
+		(instances
+			(project "SRAM_interface"
+				(path "/59b5d551-cd9e-4492-bdf8-41d0aef36030"
+					(reference "#PWR027")
+					(unit 1)
+				)
+			)
+		)
+	)
+	(symbol
+		(lib_id "power:GND")
 		(at 103.632 102.616 0)
 		(unit 1)
@@
 					(unit 1)
 				)
+			)
+		)
+	)
+	(symbol
+		(lib_id "Device:C")
+		(at 150.114 122.428 0)
+		(mirror y)
+		(unit 1)
+		(exclude_from_sim no)
+		(in_bom yes)
+		(on_board yes)
+		(dnp no)
+		(property "Reference" "C1"
+			(at 146.304 121.1579 0)
+			(effects
+				(font
+					(size 1.27 1.27)
+				)
+				(justify left)
+			)
+		)
+		(property "Value" "C"
+			(at 146.304 123.6979 0)
+			(effects
+				(font
+					(size 1.27 1.27)
+				)
+				(justify left)
+			)
+		)
+		(property "Footprint" ""
+			(at 149.1488 126.238 0)
+			(effects
+				(font
+					(size 1.27 1.27)
+				)
+				(hide yes)
+			)
+		)
+		(property "Datasheet" "~"
+			(at 150.114 122.428 0)
+			(effects
+				(font
+					(size 1.27 1.27)
+				)
+				(hide yes)
+			)
+		)
+		(property "Description" "Unpolarized capacitor"
+			(at 150.114 122.428 0)
+			(effects
+				(font
+					(size 1.27 1.27)
+				)
+				(hide yes)
+			)
+		)
+		(pin "2"
+		)
+		(pin "1"
+		)
+		(instances
+			(project ""
+				(path "/59b5d551-cd9e-4492-bdf8-41d0aef36030"
+					(reference "C1")
+					(unit 1)
+				)
